File: VECTAR-PSU-REV2.kicad_pcb (KiCad board)
At the start: 2 copper layers, 94 x 98 mm, 70 parts, among them J1 XT60PW-M, J2 XT60PW-M, J3 Conn_01x02_Socket, J5 Conn_01x06_Socket, J6 XT90PW-M, Q1 2N7002, Q3 IRFB7437, SW2 RA1113112R, U1 PLM74501QDDFRQ1, U2 PTPS543021DRLR

Commit message: Rev 2 complete - PCB and components ordered
Parts:
- removed C12, C13, C14: C, Capacitor_SMD:C_0603_1608Metric
- removed TP11: TestPoint, PSU-Rev2:KEYSTONE_5002
- added C22: 33nF, Capacitor_SMD:C_0603_1608Metric, F.Cu at (175.6, 84.4)
- C10, C21, R11, U1: moved to B.Cu
- L1: value 10uH -> 8.2uH; footprint PSU-Rev2:IND_BOURNS_SDR1307 -> PSU-Rev2:IND_BOURNS_SRP1270
- R12: value 13.7k -> 10k
- R7: value 100k -> 52.3k/1%
- R8: value 3.5k -> 52.3k/1%
- U2: value PTPS543021DRLR -> TPS62933DRLR; footprint PSU-Rev2:DRL0006A-MFG -> PSU-Rev2:SOTFL50P160X60-8N
- moved C21 156.8 mm to (134.6, 94.5), turned to -90 degrees
- moved U1 151.6 mm to (128.4, 91.7), turned to 90 degrees
- moved TP16 122.0 mm to (118.1, 50.0)
- moved TP13 76.9 mm to (188.7, 104.4), turned to 0 degrees
- moved R8 57.1 mm to (184.3, 85.5), turned to 0 degrees
- moved R2 53.2 mm to (184.3, 83.0)
- moved TP15 48.6 mm to (181.9, 103.7), turned to 0 degrees
- moved D5 48.5 mm to (193.4, 82.8), turned to 180 degrees
- moved R10 48.2 mm to (193.4, 85.2), turned to 180 degrees
- moved JP4 48.2 mm to (193.4, 87.8), turned to 180 degrees
- moved TP12 37.7 mm to (181.2, 120.7)
- moved TP4 32.6 mm to (147.2, 108.2)
- moved JP1 30.4 mm to (150.1, 108.2)
- moved JP2 30.4 mm to (152.6, 108.4)
- moved S1 30.4 mm to (154.0, 101.9)
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Connections:
- C16 pad 1: Net-(U2-BOOT) -> Net-(U2-BST)
- R2 pad 1: /Vin -> +12V
- R2 pad 2: /OV -> /5V_EN
- R8 pad 1: /OV -> /5V_EN
- U2 pad 1: +12V -> unconnected-(U2-RT-Pad1)
- U2 pad 2: Net-(U2-SW) -> /5V_EN
- U2 pad 3: GND -> +12V
- U2 pad 4: Net-(U2-BOOT) -> GND
- U2 pad 5: /5V_EN -> Net-(U2-SW)
- U2 pad 6: /5V_FB -> Net-(U2-BST)
Routing:
- net /12V_EN: track 98.5 -> 50.3 mm, vias 1 -> 2
- net +5V: track 48.0 -> 69.5 mm, vias 1 -> 2
- net +BATT: track 0.00 -> 20.9 mm, vias 0 -> 1
- net /Gate: track 0.00 -> 19.9 mm
- net /Vin_EN: track 29.0 -> 14.8 mm, vias 1 -> 0
- net Net-(U2-SW): track 11.8 -> 0.00 mm, vias 2 -> 0
- net /OV: track 8.01 -> 0.00 mm, vias 1 -> 0
- net /Vin: track 22.3 -> 30.0 mm, vias 0 -> 1
- net /RAW_BATT: track 12.2 -> 5.60 mm
- net /5V_FB: track 14.7 -> 20.9 mm, vias 0 -> 1
- net /5V_EN: track 56.3 -> 62.3 mm
- net +12V: track 5.78 -> 9.85 mm
- net Net-(U2-SS): track 0.00 -> 4.03 mm
- net Net-(U2-BST): track 0.00 -> 3.44 mm
- net Net-(U1-VCAP): track 0.00 -> 2.92 mm
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Other:
- board size 94 x 98 mm -> 94 x 85 mm
