File: VECTAR-PSU-REV2.kicad_sch (KiCad schematic)
At the start: 68 parts, among them J1 XT60PW-M, J2 XT60PW-M, J3 Conn_01x02_Socket, J5 Conn_01x06_Socket, J6 XT90PW-M, Q1 2N7002, Q3 IRFB7437, SW2 RA1113112R, U1 PLM74501QDDFRQ1, U2 PTPS543021DRLR

Commit message: Rev 2 complete - PCB and components ordered
Parts:
- removed C12, C13, C14: C, Capacitor_SMD:C_0603_1608Metric, symbol Device:C
- removed TP11: TestPoint, PSU-Rev2:KEYSTONE_5002, symbol Connector:TestPoint
- removed U2: PTPS543021DRLR, PSU-Rev2:DRL0006A-MFG, symbol PSU-Rev1:PTPS543021DRLR
- added C22: 33nF, Capacitor_SMD:C_0603_1608Metric, symbol Device:C
- added R2: 100k, Resistor_SMD:R_0603_1608Metric, symbol Device:R_US
- added R8: 52.3k/1%, Resistor_SMD:R_0603_1608Metric, symbol Device:R_US
- added U2: TPS62933DRLR, PSU-Rev2:SOTFL50P160X60-8N, symbol PSU-Rev2:TPS62933DRLR
- L1: value 10uH -> 8.2uH; footprint PSU-Rev2:IND_BOURNS_SDR1307 -> PSU-Rev2:IND_BOURNS_SRP1270
- R12: value 13.7k -> 10k
- R7: value 100k -> 52.3k/1%
Connections:
- net +12V: now also R2.1, U2.3 (VIN)
- net 5V_EN: now also R2.2, R8.1, U2.2 (EN)
- net 5V_FB: now also U2.8 (FB)
- net GND: now also C22.2, R8.2, U2.4 (GND)
- net at C16.2, L1.1: now also U2.5 (SW)
- net at C16.1: now also U2.6 (BST)
- new net: C22.1, U2.7 (SS)
- no-connect marks 0 -> 6
Other:
- moved on the sheet: C15, C16, C17, C18, C19, C20, L1, R12, R7
