File: VECTAR-PSU-REV2.kicad_sch (KiCad schematic)
At the start: 67 parts, among them J1 XT60PW-M, J2 XT60PW-M, J3 Conn_01x02_Socket, J5 Conn_01x06_Socket, J6 XT90PW-M, Q1 2N7002, Q3 IRFB7437, SW2 RA1113112R, U1 PLM74501QDDFRQ1, U2 TPS62933DRLR

Commit message: final commit
Other:
- note added: "18V Converter"
- note removed: "12V Converter"
Changed lines of the file:
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@@
 		)
 	)
-	(text "12V Converter"
+	(text "18V Converter"
 		(exclude_from_sim no)
 		(at 186.69 77.47 0)
